Commit message: simulation valid

File: src/rc_sim_description/urdf/rc_car.urdf.xacro (robot description, xacro)
@@ -8,6 +8,12 @@
   <xacro:property name="wheel_radius" value="0.06"/>
   <xacro:property name="wheel_thickness" value="0.03"/>
+  <xacro:property name="wheelbase_m" value="0.30"/>
+  <xacro:property name="rear_axle_offset_x" value="-0.15"/>
+  <xacro:property name="front_axle_offset_x" value="${rear_axle_offset_x + wheelbase_m}"/>
+  <xacro:property name="steering_limit_rad" value="0.3141592654"/>
+  <xacro:property name="lidar_offset_x" value="0.18"/>
+  <xacro:property name="lidar_offset_z" value="0.12"/>
   <!-- Placement helpers -->
-  <xacro:property name="wheel_base_x" value="${chassis_length / 2.0 - 0.07}"/>
+  <xacro:property name="wheel_base_x" value="${front_axle_offset_x}"/>
   <xacro:property name="wheel_track_y" value="${chassis_width / 2.0 + wheel_thickness / 2.0 - 0.01}"/>
   <xacro:property name="axle_height" value="${wheel_radius}"/>
@@ -89,5 +95,5 @@
       <origin xyz="${xyz}" rpy="0 0 0"/>
       <axis xyz="0 0 1"/>
-      <limit lower="-0.6" upper="0.6" effort="10.0" velocity="1.5"/>
+      <limit lower="-${steering_limit_rad}" upper="${steering_limit_rad}" effort="10.0" velocity="3.5"/>
     </joint>
     <xacro:wheel name="${name}" parent="${name}_steer" xyz="0 0 0"/>
@@ -113,5 +119,12 @@
     </collision>
   </link>
-  <link name="lidar_link">
+  <link name="rear_axle">
+    <inertial>
+      <origin xyz="0 0 0" rpy="0 0 0"/>
+      <mass value="0.02"/>
+      <inertia ixx="0.00002" ixy="0.0" ixz="0.0" iyy="0.00002" iyz="0.0" izz="0.00002"/>
+    </inertial>
+  </link>
+  <link name="laser">
     <inertial>
       <origin xyz="0 0 0" rpy="0 0 0"/>
@@ -127,4 +140,18 @@
     </visual>
   </link>
+  <link name="imu_link">
+    <inertial>
+      <origin xyz="0 0 0" rpy="0 0 0"/>
+      <mass value="0.03"/>
+      <inertia ixx="0.00005" ixy="0.0" ixz="0.0" iyy="0.00005" iyz="0.0" izz="0.00005"/>
+    </inertial>
+    <visual>
+      <origin xyz="0 0 0" rpy="0 0 0"/>
+      <geometry>
+        <box size="0.03 0.02 0.01"/>
+      </geometry>
+      <material name="chassis_grey"/>
+    </visual>
+  </link>
   <link name="camera_link">
     <inertial>
@@ -141,8 +168,21 @@
     </visual>
   </link>
+  <joint name="rear_axle_joint" type="fixed">
+    <parent link="base_link"/>
+    <child link="rear_axle"/>
+    <origin xyz="${rear_axle_offset_x} 0 ${axle_height}" rpy="0 0 0"/>
+  </joint>
   <joint name="lidar_joint" type="fixed">
     <parent link="base_link"/>
-    <child link="lidar_link"/>
-    <origin xyz="${chassis_length/2 - 0.05} 0 ${chassis_height/2 + 0.08}" rpy="0 0 0"/>
+    <child link="laser"/>
+    <origin xyz="${lidar_offset_x} 0 ${lidar_offset_z}" rpy="0 0 0"/>
+  </joint>
+  <joint name="imu_joint" type="fixed">
+    <parent link="base_link"/>
+    <child link="imu_link"/>
+    <!-- Match the real APEX planar mount: sensor Y points forward, so the
+         kinematics estimator's planar_mount_yaw_deg=-90 rotates back into
+         vehicle-forward X. -->
+    <origin xyz="0.02 0 ${chassis_height / 2.0 + 0.03}" rpy="0 0 1.57079632679"/>
   </joint>
   <joint name="camera_joint" type="fixed">
@@ -151,10 +191,10 @@
     <origin xyz="0.25 0.0 0.20" rpy="0 0 0"/>
   </joint>
-  <gazebo reference="lidar_link">
+  <gazebo reference="laser">
     <sensor name="lidar" type="gpu_lidar">
       <always_on>true</always_on>
       <update_rate>12</update_rate>
       <visualize>true</visualize>
-      <topic>/scan</topic>
+      <topic>/apex/sim/scan</topic>
       <lidar>
         <scan>
@@ -171,9 +211,54 @@
           <resolution>0.01</resolution>
         </range>
-        <noise type="gaussian">
-          <mean>0.0</mean>
-          <stddev>0.0</stddev>
-        </noise>
       </lidar>
+    </sensor>
+  </gazebo>
+  <gazebo reference="imu_link">
+    <sensor name="imu" type="imu">
+      <always_on>true</always_on>
+      <update_rate>120</update_rate>
+      <topic>/apex/sim/imu</topic>
+      <imu>
+        <angular_velocity>
+          <x>
+            <noise type="gaussian">
+              <mean>0.0</mean>
+              <stddev>0.002</stddev>
+            </noise>
+          </x>
+          <y>
+            <noise type="gaussian">
+              <mean>0.0</mean>
+              <stddev>0.002</stddev>
+            </noise>
+          </y>
+          <z>
+            <noise type="gaussian">
+              <mean>0.0</mean>
+              <stddev>0.002</stddev>
+            </noise>
+          </z>
+        </angular_velocity>
+        <linear_acceleration>
+          <x>
+            <noise type="gaussian">
+              <mean>0.0</mean>
+              <stddev>0.02</stddev>
+            </noise>
+          </x>
+          <y>
+            <noise type="gaussian">
+              <mean>0.0</mean>
+              <stddev>0.02</stddev>
+            </noise>
+          </y>
+          <z>
+            <noise type="gaussian">
+              <mean>0.0</mean>
+              <stddev>0.02</stddev>
+            </noise>
+          </z>
+        </linear_acceleration>
+      </imu>
     </sensor>
   </gazebo>
@@ -196,6 +281,4 @@
         </clip>
       </camera>
-      <frame_id>camera_link</frame_id>
-      <camera_info_topic>/camera/camera_info</camera_info_topic>
     </sensor>
   </gazebo>
@@ -204,40 +287,24 @@
   <xacro:wheel name="rear_left_wheel" parent="base_link" xyz="${-wheel_base_x} ${wheel_track_y} ${axle_height}"/>
   <xacro:wheel name="rear_right_wheel" parent="base_link" xyz="${-wheel_base_x} ${-wheel_track_y} ${axle_height}"/>
-  <ros2_control name="rc_car_system" type="system">
-    <hardware>
-      <plugin>gazebo_ros2_control/GazeboSystem</plugin>
-    </hardware>
-    <joint name="rear_left_wheel_joint">
-      <command_interface name="velocity"/>
-      <state_interface name="position"/>
-      <state_interface name="velocity"/>
-    </joint>
-    <joint name="rear_right_wheel_joint">
-      <command_interface name="velocity"/>
-      <state_interface name="position"/>
-      <state_interface name="velocity"/>
-    </joint>
-    <joint name="front_left_wheel_steer_joint">
-      <command_interface name="position"/>
-      <state_interface name="position"/>
-      <state_interface name="velocity"/>
-    </joint>
-    <joint name="front_right_wheel_steer_joint">
-      <command_interface name="position"/>
-      <state_interface name="position"/>
-      <state_interface name="velocity"/>
-    </joint>
-  </ros2_control>
-  <gazebo>
-    <plugin name="gazebo_ros2_control" filename="libgazebo_ros2_control.so"/>
-  </gazebo>
   <gazebo reference="base_link">
     <material>Gazebo/Grey</material>
-    <mu1>1.2</mu1>
-    <mu2>1.2</mu2>
-    <kp>80000.0</kp>
-    <kd>20.0</kd>
+    <mu1>1.4</mu1>
+    <mu2>1.35</mu2>
+    <kp>100000.0</kp>
+    <kd>25.0</kd>
   </gazebo>
   <gazebo>
+    <plugin
+      filename="gz-sim-joint-state-publisher-system"
+      name="gz::sim::systems::JointStatePublisher">
+    </plugin>
+    <plugin
+      filename="gz-sim-pose-publisher-system"
+      name="gz::sim::systems::PosePublisher">
+      <publish_link_pose>true</publish_link_pose>
+      <use_pose_vector_msg>true</use_pose_vector_msg>
+      <static_publisher>true</static_publisher>
+      <static_update_frequency>1</static_update_frequency>
+    </plugin>
     <plugin
       filename="gz-sim-joint-controller-system"
@@ -255,9 +322,9 @@
       <joint_name>front_left_wheel_steer_joint</joint_name>
       <topic>/model/rc_car/joint/front_left_wheel_steer_joint/cmd_pos</topic>
-      <p_gain>20.0</p_gain>
-      <i_gain>0.1</i_gain>
-      <d_gain>0.5</d_gain>
-      <cmd_max>0.6</cmd_max>
-      <cmd_min>-0.6</cmd_min>
+      <p_gain>28.0</p_gain>
+      <i_gain>0.2</i_gain>
+      <d_gain>0.7</d_gain>
+      <cmd_max>${steering_limit_rad}</cmd_max>
+      <cmd_min>-${steering_limit_rad}</cmd_min>
     </plugin>
     <plugin
@@ -266,9 +333,9 @@
       <joint_name>front_right_wheel_steer_joint</joint_name>
       <topic>/model/rc_car/joint/front_right_wheel_steer_joint/cmd_pos</topic>
-      <p_gain>20.0</p_gain>
-      <i_gain>0.1</i_gain>
-      <d_gain>0.5</d_gain>
-      <cmd_max>0.6</cmd_max>
-      <cmd_min>-0.6</cmd_min>
+      <p_gain>28.0</p_gain>
+      <i_gain>0.2</i_gain>
+      <d_gain>0.7</d_gain>
+      <cmd_max>${steering_limit_rad}</cmd_max>
+      <cmd_min>-${steering_limit_rad}</cmd_min>
     </plugin>
   </gazebo>

Commit message: Sensors error introduced

File: src/rc_sim_description/urdf/rc_car.urdf.xacro (robot description, xacro)
@@ -1,4 +1,6 @@
 <?xml version="1.0"?>
 <robot name="rc_car" xmlns:xacro="http://www.ros.org/wiki/xacro">
+  <xacro:arg name="lidar_noise_std" default="0.0"/>
+  <xacro:property name="lidar_noise_std" value="$(arg lidar_noise_std)"/>
   <!-- Basic dimensions -->
   <xacro:property name="chassis_length" value="0.46"/>
@@ -216,4 +218,10 @@
           <resolution>0.01</resolution>
         </range>
+        <!-- Optional light LiDAR noise for robustness sweeps. Default stays at
+             zero so the baseline ideal scan remains perfectly reproducible. -->
+        <noise type="gaussian">
+          <mean>0.0</mean>
+          <stddev>${lidar_noise_std}</stddev>
+        </noise>
       </lidar>
     </sensor>

Commit message: submap refiner

File: src/rc_sim_description/urdf/rc_car.urdf.xacro (robot description, xacro)
@@ -2,5 +2,9 @@
 <robot name="rc_car" xmlns:xacro="http://www.ros.org/wiki/xacro">
   <xacro:arg name="lidar_noise_std" default="0.0"/>
+  <xacro:arg name="imu_gyro_noise_stddev_rps" default="0.002"/>
+  <xacro:arg name="imu_accel_noise_stddev_mps2" default="0.02"/>
   <xacro:property name="lidar_noise_std" value="$(arg lidar_noise_std)"/>
+  <xacro:property name="imu_gyro_noise_stddev_rps" value="$(arg imu_gyro_noise_stddev_rps)"/>
+  <xacro:property name="imu_accel_noise_stddev_mps2" value="$(arg imu_accel_noise_stddev_mps2)"/>
   <!-- Basic dimensions -->
   <xacro:property name="chassis_length" value="0.46"/>
@@ -237,5 +241,5 @@
             <noise type="gaussian">
               <mean>0.0</mean>
-              <stddev>0.002</stddev>
+              <stddev>${imu_gyro_noise_stddev_rps}</stddev>
             </noise>
           </x>
@@ -243,5 +247,5 @@
             <noise type="gaussian">
               <mean>0.0</mean>
-              <stddev>0.002</stddev>
+              <stddev>${imu_gyro_noise_stddev_rps}</stddev>
             </noise>
           </y>
@@ -249,5 +253,5 @@
             <noise type="gaussian">
               <mean>0.0</mean>
-              <stddev>0.002</stddev>
+              <stddev>${imu_gyro_noise_stddev_rps}</stddev>
             </noise>
           </z>
@@ -257,5 +261,5 @@
             <noise type="gaussian">
               <mean>0.0</mean>
-              <stddev>0.02</stddev>
+              <stddev>${imu_accel_noise_stddev_mps2}</stddev>
             </noise>
           </x>
@@ -263,5 +267,5 @@
             <noise type="gaussian">
               <mean>0.0</mean>
-              <stddev>0.02</stddev>
+              <stddev>${imu_accel_noise_stddev_mps2}</stddev>
             </noise>
           </y>
@@ -269,5 +273,5 @@
             <noise type="gaussian">
               <mean>0.0</mean>
-              <stddev>0.02</stddev>
+              <stddev>${imu_accel_noise_stddev_mps2}</stddev>
             </noise>
           </z>

Commit message: RemoteTurn

File: src/rc_sim_description/urdf/rc_car.urdf.xacro (robot description, xacro)
@@ -187,8 +187,7 @@
     <parent link="base_link"/>
     <child link="imu_link"/>
-    <!-- Match the real APEX planar mount: sensor Y points forward, so the
-         kinematics estimator's planar_mount_yaw_deg=-90 rotates back into
-         vehicle-forward X. -->
-    <origin xyz="0.02 0 ${chassis_height / 2.0 + 0.03}" rpy="0 0 1.57079632679"/>
+    <!-- Match the current real APEX mount: sensor X points forward and sensor
+         Y points left, matching the vehicle base_link convention. -->
+    <origin xyz="0.02 0 ${chassis_height / 2.0 + 0.03}" rpy="0 0 0"/>
   </joint>
   <joint name="camera_joint" type="fixed">
